Commit message: added mujoco

File: robot.urdf (robot description, URDF)
Before this commit: robot C:\Users\Deepankuran M\Builds\arm, 1 links, 0 joints
Links:
- added link base_link, mass 1.0; collision mesh filename=base_link.stl; visual mesh filename=base_link.stl
- added link jaw1, mass 0.1; collision mesh filename=jaw1.stl; visual mesh filename=jaw1.stl
- added link jaw2, mass 0.1; collision mesh filename=jaw2.stl; visual mesh filename=jaw2.stl
- added link jaw3, mass 0.1; collision mesh filename=jaw3.stl; visual mesh filename=jaw3.stl
- added link jaw4, mass 0.1; collision mesh filename=jaw4.stl; visual mesh filename=jaw4.stl
- added link jaw5, mass 0.1; collision mesh filename=jaw5.stl; visual mesh filename=jaw5.stl
- added link jaw6, mass 0.1; collision mesh filename=jaw6.stl; visual mesh filename=jaw6.stl
- added link left, mass 0.3; collision mesh filename=left.stl; visual mesh filename=left.stl
- link right: mass 0.275495 -> 0.3; geometry collision mesh filename=right.stl; visual mesh filename=right.stl
Joints:
- added joint base_to_jaw1: type fixed, parent base_link, child jaw1, origin xyz=0 0 0 rpy=0 0 0
- added joint base_to_left: type fixed, parent base_link, child left, origin xyz=0 0 0 rpy=0 0 0
- added joint base_to_right: type fixed, parent base_link, child right, origin xyz=0 0 0 rpy=0 0 0
- added joint jaw1_to_jaw2: type revolute, parent jaw1, child jaw2, origin xyz=0 0 0 rpy=0 0 0, axis 0 1 0, limit lower=-1.57 upper=1.57 effort=10 velocity=1.0
- added joint jaw2_to_jaw3: type fixed, parent jaw2, child jaw3, origin xyz=0 0 0 rpy=0 0 0
- added joint jaw3_to_jaw4: type fixed, parent jaw3, child jaw4, origin xyz=0 0 0 rpy=0 0 0
- added joint jaw4_to_jaw5: type fixed, parent jaw4, child jaw5, origin xyz=0 0 0 rpy=0 0 0
- added joint jaw5_to_jaw6: type fixed, parent jaw5, child jaw6, origin xyz=0 0 0 rpy=0 0 0
